Commit message: Update irbt2005_macro.xacro

File: trackIRBT2005_support/urdf/irbt2005_macro.xacro (robot description, xacro)
@@ -8,5 +8,5 @@
         <origin xyz="0 0 0" rpy="1.5708 0 0" />
         <geometry>
-          <mesh filename="package://abb_irbt2005_support/meshes/visual/irbt2005.stl" />
+          <mesh filename="package://trackIRBT2005_support/meshes/visual/irbt2005.stl" />
         </geometry>
         <xacro:material_abb_orange/>
@@ -15,5 +15,5 @@
         <origin xyz="0 0 0" rpy="1.5708 0 0" />
         <geometry>
-          <mesh filename="package://abb_irbt2005_support/meshes/collision/irbt2005.stl" />
+          <mesh filename="package://trackIRBT2005_support/meshes/collision/irbt2005.stl" />
         </geometry>
       </collision>
@@ -23,5 +23,5 @@
         <origin xyz="0 0 0" rpy="1.5708 0 0" />
         <geometry>
-          <mesh filename="package://abb_irbt2005_support/meshes/visual/carriage_standard.stl" />
+          <mesh filename="package://trackIRBT2005_support/meshes/visual/carriage_standard.stl" />
         </geometry>
         <material name="">
@@ -32,5 +32,5 @@
         <origin xyz="0 0 0" rpy="1.5708 0 0" />
         <geometry>
-          <mesh filename="package://abb_irbt2005_support/meshes/collision/carriage_standard.stl" />
+          <mesh filename="package://trackIRBT2005_support/meshes/collision/carriage_standard.stl" />
         </geometry>
       </collision>
@@ -40,5 +40,5 @@
         <origin xyz="0 0 0" rpy="1.5708 0 0" />
         <geometry>
-          <mesh filename="package://abb_irbt2005_support/meshes/visual/carriage_mirrored.stl" />
+          <mesh filename="package://trackIRBT2005_support/meshes/visual/carriage_mirrored.stl" />
         </geometry>
         <material name="">
@@ -49,5 +49,5 @@
         <origin xyz="0 0 0" rpy="1.5708 0 0" />
         <geometry>
-          <mesh filename="package://abb_irbt2005_support/meshes/collision/carriage_mirrored.stl" />
+          <mesh filename="package://trackIRBT2005_support/meshes/collision/carriage_mirrored.stl" />
         </geometry>
       </collision>

Commit message: Update irbt2005_macro.xacro

File: trackIRBT2005_support/urdf/irbt2005_macro.xacro (robot description, xacro)
@@ -54,5 +54,5 @@
     </link>
     <!-- Joints -->
-    <joint name="${prefix}track_joint_1" type="prismatic">
+    <joint name="${prefix}track_joint1" type="prismatic">
       <origin xyz="-0.40 -0.5 -0.5" rpy="0 0 0" />
       <parent link="${prefix}track" />
@@ -61,5 +61,5 @@
       <limit lower="0" upper="5.5" effort="0" velocity="1" />
     </joint>
-    <joint name="${prefix}track_joint_2" type="prismatic">
+    <joint name="${prefix}track_joint2" type="prismatic">
       <origin xyz="-7.25 -0.5 -0.5" rpy="0 0 0" />
       <parent link="${prefix}track" />
